Commit message: v9

File: src/unitree_guide2/go1_description/xacro/robot.xacro (robot description, xacro)
@@ -125,3 +125,41 @@
         <origin rpy="0 0 0" xyz="0.2747 0.0 -0.0088"/>
     </xacro:ultraSound>
+    <link name="camera_link">
+      <visual>
+        <geometry>
+          <box size="0.02 0.02 0.02"/>
+        </geometry>
+      </visual>
+    </link>
+    <joint name="camera_joint" type="fixed">
+      <parent link="trunk"/>
+      <child link="camera_link"/>
+      <origin xyz="0.21 0 0.25" rpy="0 0 0"/>
+    </joint>
+    <gazebo reference="camera_link">
+      <sensor name="camera" type="depth">
+        <update_rate>15</update_rate>
+        <camera>
+          <horizontal_fov>1.0</horizontal_fov>
+          <image>
+            <width>320</width>
+            <height>240</height>
+            <format>R8G8B8</format>
+          </image>
+          <clip>
+            <near>0.1</near>
+            <far>5.0</far>
+          </clip>
+        </camera>
+        <plugin name="gazebo_ros_camera" filename="libgazebo_ros_camera.so">
+          <ros>
+            <namespace>/camera</namespace>
+          </ros>
+          <frame_name>camera_link</frame_name>
+          <image_topic_name>image_raw</image_topic_name>
+          <depth_image_topic_name>depth/image_raw</depth_image_topic_name>
+          <point_cloud_topic_name>points</point_cloud_topic_name>
+        </plugin>
+      </sensor>
+    </gazebo>
 </robot>

Commit message: v10

File: src/unitree_guide2/go1_description/xacro/robot.xacro (robot description, xacro)
@@ -137,29 +137,35 @@
       <origin xyz="0.21 0 0.25" rpy="0 0 0"/>
     </joint>
+    <link name="camera_optical_frame"/>
+    <joint name="camera_optical_joint" type="fixed">
+      <parent link="camera_link"/>
+      <child link="camera_optical_frame"/>
+      <origin xyz="0 0 0" rpy="-1.5708 0 -1.5708"/>
+    </joint>
     <gazebo reference="camera_link">
-      <sensor name="camera" type="depth">
-        <update_rate>15</update_rate>
-        <camera>
-          <horizontal_fov>1.0</horizontal_fov>
-          <image>
-            <width>320</width>
-            <height>240</height>
-            <format>R8G8B8</format>
-          </image>
-          <clip>
-            <near>0.1</near>
-            <far>5.0</far>
-          </clip>
-        </camera>
-        <plugin name="gazebo_ros_camera" filename="libgazebo_ros_camera.so">
-          <ros>
-            <namespace>/camera</namespace>
-          </ros>
-          <frame_name>camera_link</frame_name>
-          <image_topic_name>image_raw</image_topic_name>
-          <depth_image_topic_name>depth/image_raw</depth_image_topic_name>
-          <point_cloud_topic_name>points</point_cloud_topic_name>
-        </plugin>
-      </sensor>
-    </gazebo>
+  <sensor name="camera" type="depth">
+    <update_rate>30</update_rate>
+    <camera>
+      <horizontal_fov>1.0</horizontal_fov>
+      <image>
+        <width>640</width>
+        <height>480</height>
+        <format>R8G8B8</format>
+      </image>
+      <clip>
+        <near>0.3</near>
+        <far>3.0</far>
+      </clip>
+    </camera>
+    <plugin name="gazebo_ros_camera" filename="libgazebo_ros_camera.so">
+      <ros>
+        <namespace>/camera</namespace>
+      </ros>
+      <frame_name>camera_optical_frame</frame_name>
+      <image_topic_name>image_raw</image_topic_name>
+      <depth_image_topic_name>depth/image_raw</depth_image_topic_name>
+      <point_cloud_topic_name>points</point_cloud_topic_name>
+    </plugin>
+  </sensor>
+</gazebo>
 </robot>

Commit message: v11

File: src/unitree_guide2/go1_description/xacro/robot.xacro (robot description, xacro)
@@ -135,5 +135,5 @@
       <parent link="trunk"/>
       <child link="camera_link"/>
-      <origin xyz="0.21 0 0.25" rpy="0 0 0"/>
+      <origin xyz="0.26 0 0.1" rpy="0 0 0"/>
     </joint>
     <link name="camera_optical_frame"/>
